Commit message: simulation working with gripper and rviz file

File: tictactoe-bot/src/end_effector/urdf/my_gripper.urdf (robot description, URDF)
Before this commit: robot my_gripper, 1 links, 0 joints
Links:
- link gripper_base_link: geometry collision box size=0.06 0.1 0.03; visual mesh filename=package://end_effector/meshes/GripperViz.stl scale=0.001 0.001 0.001
